Commit message: fixed arm falling

File: Simulation/ArmObj/Robot_Arm.urdf (robot description, URDF)
Before this commit: robot simple_claw_robot, 14 links, 13 joints
Links:
- added link Camera, mass 0.001; collision mesh filename=Camera.obj; visual mesh filename=Camera.obj
- added link Camera_Arm, mass 0.123; collision mesh filename=Camera_Arm.obj; visual mesh filename=Camera_Arm.obj
- added link Camera_Mount, mass 0.001; collision mesh filename=Camera_Mount.obj; visual mesh filename=Camera_Mount.obj
- added link Claw_PadL, mass 0.001; collision mesh filename=Claw_PadL.obj; visual mesh filename=Claw_PadL.obj
- added link Claw_PadR, mass 0.001; collision mesh filename=Claw_PadR.obj; visual mesh filename=Claw_PadR.obj
- added link Lidar_Base, mass 0.001; collision mesh filename=Lidar_Base.obj; visual mesh filename=Lidar_Base.obj
- added link Lidar_Lense, mass 0.001; collision mesh filename=Lidar_Lense.obj; visual mesh filename=Lidar_Lense.obj
Joints:
- added joint BaseWoodtoCameraArm: type revolute, parent Base_Wood, child Camera_Arm, origin xyz=0.123 -0.215 0.0075 rpy=0 0 0, axis 0.0 0.0 1.0, limit lower=-1.57 upper=1.57 effort=1.0 velocity=1.0
- added joint CameraArmtoCameraMount: type revolute, parent Camera_Arm, child Camera_Mount, origin xyz=0.0 0.0 0.45 rpy=0 0 0, axis 1.0 0.0 0.0, limit lower=-1.57 upper=1.57 effort=1.0 velocity=1.0
- added joint CameraMounttoCamera: type fixed, parent Camera_Mount, child Camera, origin xyz=0.0 0.0025 0.03 rpy=0 0 0
- added joint ClawLefttoClawPad: type fixed, parent Claw_Left, child Claw_PadL, origin xyz=-0.0145 0.0 0.08 rpy=0 0 0
- added joint ClawRighttoClawPad: type fixed, parent Claw_Right, child Claw_PadR, origin xyz=0.0145 0.0 0.08 rpy=0 0 0
- added joint ClawServotoLidarBase: type fixed, parent Claw_Servo, child Lidar_Base, origin xyz=0.0125 0.005 0.0125 rpy=0 0 0
- added joint LidarBasetoLidarLense: type fixed, parent Lidar_Base, child Lidar_Lense, origin xyz=0.0 0.0 0.0075 rpy=0 0 0
- joint ClawBasetoClawLeft: origin xyz=-0.025 0.0 0.03 rpy=0 0 0 -> xyz=0.005 0.0 0.03 rpy=0 0 0; type fixed -> revolute
- joint ClawBasetoClawRight: origin xyz=0.005 0.0 0.03 rpy=0 0 0 -> xyz=-0.025 0.0 0.03 rpy=0 0 0; type fixed -> revolute
- joint ShouldertoBracket: limit lower=-1.57 upper=1.57 effort=1.0 velocity=1.0 -> lower=-1.57 upper=1.57 effort=100.0 velocity=0.0
